File: hardware/kiCad/Mercury/Mercury.kicad_pcb (KiCad board)
At the start: 4 copper layers, 5.1 x 8.1 mm, 124 parts, among them J1 SWD, J10 OUTPUT, J11 Analog I/O, J12 Power Rails, J13 5-1814832-1, J14 5-1814832-1, J2 I2C1, J3 I2C2, J4 UART1, J5 SPI1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

Commit message: Refresh
Parts:
- removed R24, R25: 22, Resistor_SMD:R_0402_1005Metric
- H1, H2, H3, H4: footprint MountingHole:MountingHole_4.3mm_M4_Pad_Via -> MountingHole:MountingHole_3mm_Pad_Via
- J2: value I2C1 -> UART1; footprint Connector_Wire:SolderWire-0.25sqmm_1x04_P4.2mm_D0.65mm_OD1.7mm -> Connector_Wire:SolderWire-0.1sqmm_1x02_P3.6mm_D0.4mm_OD1mm
- J3, J5, J6: footprint Connector_Wire:SolderWire-0.25sqmm_1x06_P4.2mm_D0.65mm_OD1.7mm -> Connector_Wire:SolderWire-0.1sqmm_1x04_P3.6mm_D0.4mm_OD1mm
- J4: footprint Connector_Wire:SolderWire-0.25sqmm_1x04_P4.2mm_D0.65mm_OD1.7mm -> Connector_Wire:SolderWire-0.1sqmm_1x02_P3.6mm_D0.4mm_OD1mm
- moved H2 122.4 mm to (116.4, 23.8)
- moved H4 112.5 mm to (24.0, 96.2)
- moved C27 84.0 mm to (99.7, -8.33)
- moved C29 84.0 mm to (95.2, -11.0)
- moved C30 84.0 mm to (95.1, -12.0)
- moved C31 84.0 mm to (98.4, -16.1)
- moved C32 84.0 mm to (97.4, -16.1)
- moved C34 84.0 mm to (106.6, -8.07)
- moved C35 84.0 mm to (106.3, -15.7)
- moved C36 84.0 mm to (97.8, -25.1)
- moved C37 84.0 mm to (97.8, -23.8)
- moved C41 84.0 mm to (102.6, -26.1)
- moved C42 84.0 mm to (92.8, -25.3)
- moved C43 84.0 mm to (105.0, -29.2)
- moved C44 84.0 mm to (94.3, -21.8)
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Connections:
- J2 pad 1: +3V3 -> Net-(J2-Pad1)
- J3 pad 1: +3V3 -> Net-(J3-Pad1)
- J4 pad 1: +3V3 -> Net-(J4-Pad1)
- J5 pad 1: +3V3 -> Net-(J5-Pad1)
- J6 pad 1: +3V3 -> Net-(J6-Pad1)
- J7 pad 2: Net-(J7-Pad2) -> USB_D-
- J7 pad 3: Net-(J7-Pad3) -> USB_D+
- R14 pad 2: Net-(J4-Pad2) -> Net-(J4-Pad1)
- R15 pad 2: Net-(J4-Pad3) -> Net-(J4-Pad2)
- R16 pad 2: Net-(J5-Pad2) -> Net-(J5-Pad1)
- R17 pad 2: Net-(J5-Pad3) -> Net-(J5-Pad2)
- R18 pad 2: Net-(J5-Pad4) -> Net-(J5-Pad3)
- R19 pad 2: Net-(J5-Pad5) -> Net-(J5-Pad4)
- R20 pad 1: SPI2_SCK -> SPI2_MOSI
- R20 pad 2: Net-(J6-Pad2) -> Net-(J6-Pad1)
- R21 pad 1: SPI2_MISO -> SPI2_SCK
- R21 pad 2: Net-(J6-Pad3) -> Net-(J6-Pad2)
- R22 pad 1: SPI2_MOSI -> FLASH_CS
- R22 pad 2: Net-(J6-Pad4) -> Net-(J6-Pad3)
- R23 pad 1: FLASH_CS -> SPI2_MISO
- R23 pad 2: Net-(J6-Pad5) -> Net-(J6-Pad4)
- R4 pad 1: I2C1_SCL -> I2C1_SDA
- R4 pad 2: Net-(J2-Pad2) -> Net-(J2-Pad1)
- R5 pad 1: I2C1_SDA -> I2C1_SCL
- R5 pad 2: Net-(J2-Pad3) -> Net-(J2-Pad2)
- R6 pad 2: Net-(J3-Pad2) -> Net-(J3-Pad1)
- R7 pad 2: Net-(J3-Pad3) -> Net-(J3-Pad2)
- R8 pad 1: ALT_INT_2 -> ALT_INT_1
- R8 pad 2: Net-(J3-Pad4) -> Net-(J3-Pad3)
- R9 pad 1: ALT_INT_1 -> ALT_INT_2
- R9 pad 2: Net-(J3-Pad5) -> Net-(J3-Pad4)
- U1 pad 2: Net-(U1-Pad2) -> ~GPS_RESET
- U1 pad 3: Net-(U1-Pad3) -> GPS_LNA_EN
- U1 pad 4: Net-(U1-Pad4) -> TIME_PULSE
- U1 pad 5: Net-(U1-Pad5) -> ~GPS_SAFEBOOT
- U1 pad 64: ~GPS_SAFEBOOT -> Net-(U1-Pad64)
- U1 pad 65: GPS_LNA_EN -> Net-(U1-Pad65)
- U1 pad 66: TIME_PULSE -> Net-(U1-Pad66)
- U1 pad 67: ~GPS_RESET -> Net-(U1-Pad67)
Other:
- board size 5.1 x 8.1 mm -> 100 x 80 mm

Commit message: Layout Done
Parts:
- removed C24: 100nF, Capacitor_SMD:C_0402_1005Metric
- removed R9: 22, Resistor_SMD:R_0402_1005Metric
- C25: value 10uF -> 4.7uF
- J3: footprint Connector_Wire:SolderWire-0.1sqmm_1x04_P3.6mm_D0.4mm_OD1mm -> Connector_Wire:SolderWire-0.1sqmm_1x03_P3.6mm_D0.4mm_OD1mm
- J8: footprint TerminalBlock_Phoenix:TerminalBlock_Phoenix_MKDS-3-2-5.08_1x02_P5.08mm_Horizontal -> TerminalBlock_Phoenix:TerminalBlock_Phoenix_MKDS-1,5-2-5.08_1x02_P5.08mm_Horizontal
- U6: value MPL3115A2 -> LPS25HB; footprint Package_LGA:NXP_LGA-8_3x5mm_P1.25mm_H1.1mm -> Package_LGA:ST_HLGA-10_2.5x2.5mm_P0.6mm_LayoutBorder3x2y
- moved J14 72.0 mm to (115.2, 36.1), turned to 180 degrees
- moved C43 65.5 mm to (108.1, 36.3)
- moved L4 64.5 mm to (106.3, 35.8), turned to 0 degrees
- moved C35 62.2 mm to (89.4, 44.2), turned to 270 degrees
- moved R35 62.1 mm to (87.1, 40.8), turned to 270 degrees
- moved L2 61.9 mm to (99.7, 35.8)
- moved C42 61.7 mm to (104.6, 35.3)
- moved R36 61.7 mm to (96.8, 39.4), turned to 270 degrees
- moved C41 61.4 mm to (101.4, 35.3), turned to 270 degrees
- moved L3 60.9 mm to (103.1, 35.8), turned to 0 degrees
- moved Y2 60.0 mm to (85.9, 44.1), turned to 0 degrees
- moved C44 59.7 mm to (109.7, 35.8), turned to 180 degrees
- moved C32 58.1 mm to (86.0, 40.8), turned to 270 degrees
- moved C34 57.3 mm to (82.5, 43.9), turned to 90 degrees
- moved U8 56.5 mm to (95.8, 35.4), turned to 0 degrees
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Connections:
- C28 pad 1: Net-(C28-Pad1) -> +3V3
- C29 pad 1: Net-(C28-Pad1) -> +3V3
- C30 pad 1: Net-(C28-Pad1) -> +3V3
- C31 pad 1: Net-(C28-Pad1) -> +3V3
- C32 pad 1: Net-(C28-Pad1) -> +3V3
- R16 pad 1: SPI1_SCK -> RF_CS
- R18 pad 1: SPI1_MOSI -> SPI1_SCK
- R19 pad 1: RF_CS -> SPI1_MOSI
- U1 pad 45: ALT_INT_2 -> Net-(U1-Pad45)
- U6 pad 2: V_CAP_ALT -> I2C2_SCL
- U6 pad 4: +3V3 -> I2C2_SDA
- U6 pad 5: ALT_INT_2 -> GND
- U6 pad 6: ALT_INT_1 -> GND
- U6 pad 7: I2C2_SDA -> ALT_INT_1
- U6 pad 8: I2C2_SCL -> GND

Commit message: Added USB
Parts:
- J7: value 629105150521 -> 1981568-1; footprint 629105150521:629105150521 -> USB:1981568-1
- moved J7 2.27 mm to (20.3, 62.5)

Commit message: Layout + Routing v1 done
Parts:
- moved C20 18.0 mm to (81.8, 83.6), turned to 0 degrees
- moved C19 16.9 mm to (78.2, 86.4), turned to 270 degrees
- moved C21 15.5 mm to (76.5, 86.4), turned to 270 degrees
- moved J2 10.5 mm to (72.2, 74.1), turned to 0 degrees
- moved U4 9.76 mm to (77.6, 82.4), turned to 0 degrees
- moved C22 8.94 mm to (78.3, 77.8), turned to 90 degrees
- moved C13 7.12 mm to (85.3, 63.2), turned to 180 degrees
- moved C14 6.63 mm to (85.1, 56.7), turned to 0 degrees
- moved R5 6.23 mm to (76.1, 76.7), turned to 90 degrees
- moved R4 6.10 mm to (72.0, 76.7), turned to 90 degrees
- moved J1 5.04 mm to (22.2, 80.7), turned to 0 degrees
- moved R27 4.97 mm to (71.6, 78.4), turned to 0 degrees
- moved R10 4.61 mm to (27.5, 86.0)
- moved R13 4.33 mm to (27.9, 80.7)
- moved R26 3.21 mm to (75.5, 78.5), turned to 0 degrees
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Connections:
- C36 pad 2: Net-(C36-Pad2) -> GND
- C37 pad 2: Net-(C36-Pad2) -> GND
- J11 pad 1: AGPIO1 -> AGPIO2
- J11 pad 2: AGPIO2 -> AGPIO1
Routing:
- net GND: track 0.00 -> 292.4 mm, vias 0 -> 145
- net +3V3: track 0.00 -> 183.0 mm, vias 0 -> 76
- net NRST: track 0.00 -> 56.5 mm
- net UART1_RX: track 0.00 -> 54.0 mm, vias 0 -> 2
- net SWO: track 0.00 -> 49.1 mm, vias 0 -> 2
- net UART1_TX: track 0.00 -> 48.8 mm, vias 0 -> 2
- net ~GPS_SAFEBOOT: track 0.00 -> 45.8 mm, vias 0 -> 2
- net SWDIO: track 0.00 -> 43.6 mm, vias 0 -> 2
- net AGPIO2: track 0.00 -> 42.8 mm
- net SWCLK: track 0.00 -> 41.4 mm
- net RF_HGM: track 0.00 -> 40.5 mm, vias 0 -> 4
- net RF_LNA_EN: track 0.00 -> 39.7 mm
- net RF_PA_EN: track 0.00 -> 39.4 mm, vias 0 -> 2
- net AGPIO1: track 0.00 -> 38.7 mm
- net GPS_LNA_EN: track 0.00 -> 38.5 mm
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- added copper zone on In2.Cu, net +3V3
- added copper zone on B.Cu, net GND
- added copper zone on F.Cu, net GND
- added copper zone on In1.Cu, net GND

Commit message: Updated with final board design
Parts:
- added G***: LOGO, LOGO:LOGO, F.Cu at (106.4, 49.7)
- moved R29 17.1 mm to (57.2, 43.8)
- moved R28 16.7 mm to (59.1, 43.9), turned to 180 degrees
- moved R1 1.75 mm to (85.8, 92.0)
- moved SW1 1.75 mm to (84.3, 97.7)
- moved R15 1.02 mm to (108.5, 72.0), turned to 180 degrees
- moved J8 0.12 mm to (25.9, 42.6)
Connections:
- U6 pad 6: GND -> +3V3
Routing:
- net GND: track 292.4 -> 356.9 mm, vias 145 -> 382
- net UART1_RX: track 54.0 -> 62.4 mm
- net Vin: track 13.0 -> 19.7 mm
- net +3V3: track 183.0 -> 185.8 mm, vias 76 -> 77
- net UART1_TX: track 48.8 -> 51.7 mm
- net RF_GPO1: track 34.7 -> 32.0 mm
- net RF_CS: track 28.9 -> 27.1 mm
- net RF_LNA_EN: track 39.7 -> 41.4 mm, vias 0 -> 2
- net I2C1_SCL: track 16.8 -> 18.3 mm
- net I2C2_SDA: track 32.9 -> 34.2 mm
- net ALT_INT_1: track 36.1 -> 34.8 mm
- net I2C1_SDA: track 17.2 -> 18.1 mm
- net BOOT0: track 32.9 -> 33.7 mm
- net I2C2_SCL: track 32.5 -> 33.0 mm
- net (no net): vias 0 -> 2
