File: hardware/kiCad/Mercury/Mercury.sch (KiCad schematic (older format))
At the start: 72 parts, among them J1 SWD, J10 OUTPUT, J11 Analog I/O, J12 Power Rails, J2 UART1, J3 I2C2, J4 UART1, J5 SPI1, J6 SPI2, J7 1981568-1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

Commit message: Updated with final board design
Other:
- moved on the sheet: H1, H2, H3, H4
Changed lines of the file:
@@
 L Mechanical:MountingHole_Pad H1
 U 1 1 5FF0F3E1
-P 8450 4100
-F 0 "H1" V 8404 4250 50  0000 L CNN
-F 1 "MountingHole_Pad" V 8495 4250 50  0000 L CNN
-F 2 "MountingHole:MountingHole_3mm_Pad_Via" H 8450 4100 50  0001 C CNN
-F 3 "~" H 8450 4100 50  0001 C CNN
-	1    8450 4100
+P 8850 3950
+F 0 "H1" V 8804 4100 50  0000 L CNN
+F 1 "MountingHole_Pad" V 8895 4100 50  0000 L CNN
+F 2 "MountingHole:MountingHole_3mm_Pad_Via" H 8850 3950 50  0001 C CNN
+F 3 "~" H 8850 3950 50  0001 C CNN
+	1    8850 3950
 	0    1    1    0
 $EndComp
@@
 L Mechanical:MountingHole_Pad H2
 U 1 1 5FF1023E
-P 8450 4325
-F 0 "H2" V 8404 4475 50  0000 L CNN
-F 1 "MountingHole_Pad" V 8495 4475 50  0000 L CNN
-F 2 "MountingHole:MountingHole_3mm_Pad_Via" H 8450 4325 50  0001 C CNN
-F 3 "~" H 8450 4325 50  0001 C CNN
-	1    8450 4325
+P 8850 4175
+F 0 "H2" V 8804 4325 50  0000 L CNN
+F 1 "MountingHole_Pad" V 8895 4325 50  0000 L CNN
+F 2 "MountingHole:MountingHole_3mm_Pad_Via" H 8850 4175 50  0001 C CNN
+F 3 "~" H 8850 4175 50  0001 C CNN
+	1    8850 4175
 	0    1    1    0
 $EndComp
@@
 L Mechanical:MountingHole_Pad H3
 U 1 1 5FF10974
-P 8450 4575
-F 0 "H3" V 8404 4725 50  0000 L CNN
-F 1 "MountingHole_Pad" V 8495 4725 50  0000 L CNN
-F 2 "MountingHole:MountingHole_3mm_Pad_Via" H 8450 4575 50  0001 C CNN
-F 3 "~" H 8450 4575 50  0001 C CNN
-	1    8450 4575
+P 8850 4425
+F 0 "H3" V 8804 4575 50  0000 L CNN
+F 1 "MountingHole_Pad" V 8895 4575 50  0000 L CNN
+F 2 "MountingHole:MountingHole_3mm_Pad_Via" H 8850 4425 50  0001 C CNN
+F 3 "~" H 8850 4425 50  0001 C CNN
+	1    8850 4425
 	0    1    1    0
 $EndComp
@@
 L Mechanical:MountingHole_Pad H4
 U 1 1 5FF11360
-P 8450 4800
-F 0 "H4" V 8404 4950 50  0000 L CNN
-F 1 "MountingHole_Pad" V 8495 4950 50  0000 L CNN
-F 2 "MountingHole:MountingHole_3mm_Pad_Via" H 8450 4800 50  0001 C CNN
-F 3 "~" H 8450 4800 50  0001 C CNN
-	1    8450 4800
+P 8850 4650
+F 0 "H4" V 8804 4800 50  0000 L CNN
+F 1 "MountingHole_Pad" V 8895 4800 50  0000 L CNN
+F 2 "MountingHole:MountingHole_3mm_Pad_Via" H 8850 4650 50  0001 C CNN
+F 3 "~" H 8850 4650 50  0001 C CNN
+	1    8850 4650
 	0    1    1    0
 $EndComp
@@
 L power:GND #PWR0189
 U 1 1 5FF19494
-P 8350 4100
-F 0 "#PWR0189" H 8350 3850 50  0001 C CNN
-F 1 "GND" H 8200 4050 50  0001 C CNN
-F 2 "" H 8350 4100 50  0001 C CNN
-F 3 "" H 8350 4100 50  0001 C CNN
-	1    8350 4100
+P 8750 3950
+F 0 "#PWR0189" H 8750 3700 50  0001 C CNN
+F 1 "GND" H 8600 3900 50  0001 C CNN
+F 2 "" H 8750 3950 50  0001 C CNN
+F 3 "" H 8750 3950 50  0001 C CNN
+	1    8750 3950
 	0    1    1    0
 $EndComp
@@
 L power:GND #PWR0190
 U 1 1 5FF1A7DD
-P 8350 4325
-F 0 "#PWR0190" H 8350 4075 50  0001 C CNN
-F 1 "GND" H 8200 4275 50  0001 C CNN
-F 2 "" H 8350 4325 50  0001 C CNN
-F 3 "" H 8350 4325 50  0001 C CNN
-	1    8350 4325
+P 8750 4175
+F 0 "#PWR0190" H 8750 3925 50  0001 C CNN
+F 1 "GND" H 8600 4125 50  0001 C CNN
+F 2 "" H 8750 4175 50  0001 C CNN
+F 3 "" H 8750 4175 50  0001 C CNN
+	1    8750 4175
 	0    1    1    0
 $EndComp
@@
 L power:GND #PWR0191
 U 1 1 5FF1ABD3
-P 8350 4575
-F 0 "#PWR0191" H 8350 4325 50  0001 C CNN
-F 1 "GND" H 8200 4525 50  0001 C CNN
-F 2 "" H 8350 4575 50  0001 C CNN
-F 3 "" H 8350 4575 50  0001 C CNN
-	1    8350 4575
+P 8750 4425
+F 0 "#PWR0191" H 8750 4175 50  0001 C CNN
+F 1 "GND" H 8600 4375 50  0001 C CNN
+F 2 "" H 8750 4425 50  0001 C CNN
+F 3 "" H 8750 4425 50  0001 C CNN
+	1    8750 4425
 	0    1    1    0
 $EndComp
@@
 L power:GND #PWR0192
 U 1 1 5FF1AF62
-P 8350 4800
-F 0 "#PWR0192" H 8350 4550 50  0001 C CNN
-F 1 "GND" H 8200 4750 50  0001 C CNN
-F 2 "" H 8350 4800 50  0001 C CNN
-F 3 "" H 8350 4800 50  0001 C CNN
-	1    8350 4800
+P 8750 4650
+F 0 "#PWR0192" H 8750 4400 50  0001 C CNN
+F 1 "GND" H 8600 4600 50  0001 C CNN
+F 2 "" H 8750 4650 50  0001 C CNN
+F 3 "" H 8750 4650 50  0001 C CNN
+	1    8750 4650
 	0    1    1    0
 $EndComp
