File: hardware/kiCad/Mercury/peripherals.sch (KiCad schematic (older format))
At the start: 49 parts, among them J13 5-1814832-1, J14 5-1814832-1, U4 MPU-6050, U5 W25N01GVZEIG_TR, U6 MPL3115A2, U7 CC2500, U8 CC2592RGVR, U9 MAX-8Q, Y2 26 MHz Oscillator

Commit message: Layout Done
Parts:
- removed C24: 100nF, Capacitor_SMD:C_0402_1005Metric, symbol Device:C_Small
- removed U6: MPL3115A2, Package_LGA:NXP_LGA-8_3x5mm_P1.25mm_H1.1mm, symbol Sensor_Pressure:MPL3115A2
- added U6: LPS25HB, Package_LGA:ST_HLGA-10_2.5x2.5mm_P0.6mm_LayoutBorder3x2y, symbol Sensor_Pressure:LPS25HB
- C25: value 10uF -> 4.7uF
Connections:
- net labels removed: ALT_INT_2, V_CAP_ALT
- wire segments 102 -> 100
Other:
- moved on the sheet: C25, C26
Changed lines of the file:
@@
 Wire Wire Line
 	6850 1700 6825 1700
-$Comp
-L Sensor_Pressure:MPL3115A2 U6
-U 1 1 5FEBCDEA
-P 7925 1550
-F 0 "U6" H 7675 2000 50  0000 C CNN
-F 1 "MPL3115A2" H 8175 2025 50  0000 C CNN
-F 2 "Package_LGA:NXP_LGA-8_3x5mm_P1.25mm_H1.1mm" H 8925 1100 50  0001 C CNN
-F 3 "https://www.nxp.com/docs/en/data-sheet/MPL3115A2.pdf" H 7925 1550 50  0001 C CNN
-	1    7925 1550
-	1    0    0    -1
-$EndComp
-Text GLabel 8325 1450 2    50   Input ~ 0
+Text GLabel 8100 1875 3    50   Input ~ 0
 ALT_INT_1
-Text GLabel 8325 1550 2    50   Input ~ 0
-ALT_INT_2
-Text GLabel 7525 1450 0    50   Input ~ 0
+Text GLabel 8600 1875 3    50   Input ~ 0
 I2C2_SDA
-Text GLabel 7525 1550 0    50   Input ~ 0
+Text GLabel 8400 1875 3    50   Input ~ 0
 I2C2_SCL
-Text GLabel 8325 1750 2    50   Input ~ 0
-V_CAP_ALT
-Text GLabel 9025 1300 2    50   Input ~ 0
-V_CAP_ALT
 $Comp
 L power:GND #PWR0152
 U 1 1 5FEC1E70
-P 7925 2050
-F 0 "#PWR0152" H 7925 1800 50  0001 C CNN
-F 1 "GND" H 7930 1877 50  0000 C CNN
-F 2 "" H 7925 2050 50  0001 C CNN
-F 3 "" H 7925 2050 50  0001 C CNN
-	1    7925 2050
-	1    0    0    -1
-$EndComp
-$Comp
-L Device:C_Small C24
-U 1 1 5FEC2756
-P 8975 1475
-F 0 "C24" H 9067 1521 50  0000 L CNN
-F 1 "100nF" H 9067 1430 50  0000 L CNN
-F 2 "Capacitor_SMD:C_0402_1005Metric" H 8975 1475 50  0001 C CNN
-F 3 "~" H 8975 1475 50  0001 C CNN
-	1    8975 1475
-	1    0    0    -1
-$EndComp
-$Comp
-L power:GND #PWR0153
-U 1 1 5FEC37C3
-P 8975 1650
-F 0 "#PWR0153" H 8975 1400 50  0001 C CNN
-F 1 "GND" H 8980 1477 50  0000 C CNN
-F 2 "" H 8975 1650 50  0001 C CNN
-F 3 "" H 8975 1650 50  0001 C CNN
-	1    8975 1650
-	1    0    0    -1
-$EndComp
-Wire Wire Line
-	8975 1575 8975 1650
-Wire Wire Line
-	8975 1375 8975 1300
-Wire Wire Line
-	8975 1300 9025 1300
+P 7900 1275
+F 0 "#PWR0152" H 7900 1025 50  0001 C CNN
+F 1 "GND" H 7905 1102 50  0000 C CNN
+F 2 "" H 7900 1275 50  0001 C CNN
+F 3 "" H 7900 1275 50  0001 C CNN
+	1    7900 1275
+	1    0    0    -1
+$EndComp
 Text GLabel 3325 600  2    50   Input ~ 0
 IMU_CAP_OUT
@@
 $EndComp
 $Comp
-L Device:C_Small C26
-U 1 1 5FEC6044
-P 9900 1550
-F 0 "C26" H 9992 1596 50  0000 L CNN
-F 1 "100nF" H 9992 1505 50  0000 L CNN
-F 2 "Capacitor_SMD:C_0603_1608Metric" H 9900 1550 50  0001 C CNN
-F 3 "~" H 9900 1550 50  0001 C CNN
-	1    9900 1550
-	1    0    0    -1
-$EndComp
-$Comp
-L power:GND #PWR0155
-U 1 1 5FEC6232
-P 9900 1650
-F 0 "#PWR0155" H 9900 1400 50  0001 C CNN
-F 1 "GND" H 9905 1477 50  0000 C CNN
-F 2 "" H 9900 1650 50  0001 C CNN
-F 3 "" H 9900 1650 50  0001 C CNN
-	1    9900 1650
-	1    0    0    -1
-$EndComp
-$Comp
 L power:+3.3V #PWR0156
 U 1 1 5FEC623C
-P 9900 1450
-F 0 "#PWR0156" H 9900 1300 50  0001 C CNN
-F 1 "+3.3V" H 9915 1623 50  0000 C CNN
-F 2 "" H 9900 1450 50  0001 C CNN
-F 3 "" H 9900 1450 50  0001 C CNN
-	1    9900 1450
-	1    0    0    -1
-$EndComp
-$Comp
-L Device:C_Small C25
-U 1 1 5FEC8637
-P 9650 1550
-F 0 "C25" H 9450 1600 50  0000 L CNN
-F 1 "10uF" H 9400 1500 50  0000 L CNN
-F 2 "Capacitor_SMD:C_0805_2012Metric" H 9650 1550 50  0001 C CNN
-F 3 "~" H 9650 1550 50  0001 C CNN
-	1    9650 1550
-	1    0    0    -1
-$EndComp
-Wire Wire Line
-	9650 1450 9900 1450
-Connection ~ 9900 1450
-Wire Wire Line
-	9650 1650 9900 1650
-Connection ~ 9900 1650
-$Comp
-L power:+3.3V #PWR0157
-U 1 1 5FECC0FE
-P 7925 1025
-F 0 "#PWR0157" H 7925 875 50  0001 C CNN
-F 1 "+3.3V" H 7940 1198 50  0000 C CNN
-F 2 "" H 7925 1025 50  0001 C CNN
-F 3 "" H 7925 1025 50  0001 C CNN
-	1    7925 1025
-	1    0    0    -1
-$EndComp
-Wire Wire Line
-	7925 1025 7925 1050
-Wire Wire Line
-	7925 1025 7825 1025
-Wire Wire Line
-	7825 1025 7825 1050
-Connection ~ 7925 1025
+P 8900 1175
+F 0 "#PWR0156" H 8900 1025 50  0001 C CNN
+F 1 "+3.3V" H 8915 1348 50  0000 C CNN
+F 2 "" H 8900 1175 50  0001 C CNN
+F 3 "" H 8900 1175 50  0001 C CNN
+	1    8900 1175
+	1    0    0    -1
+$EndComp
 Wire Wire Line
 	1700 900  1700 925
@@
 L power:+3.3V #PWR0183
 U 1 1 5FECDC32
-P 1200 2825
-F 0 "#PWR0183" H 1200 2675 50  0001 C CNN
-F 1 "+3.3V" H 1215 2998 50  0000 C CNN
-F 2 "" H 1200 2825 50  0001 C CNN
-F 3 "" H 1200 2825 50  0001 C CNN
-	1    1200 2825
+P 1200 2800
+F 0 "#PWR0183" H 1200 2650 50  0001 C CNN
+F 1 "+3.3V" H 1215 2973 50  0000 C CNN
+F 2 "" H 1200 2800 50  0001 C CNN
+F 3 "" H 1200 2800 50  0001 C CNN
+	1    1200 2800
 	1    0    0    -1
 $EndComp
@@
 $EndComp
 Wire Wire Line
-	1200 2800 1600 2800
-Wire Wire Line
 	1600 3025 2000 3025
 Wire Wire Line
@@
 Wire Wire Line
 	2000 2800 2000 2825
-Connection ~ 1600 2800
 $Comp
 L Device:C_Small C30
@@
 	1    0    0    -1
 $EndComp
+Wire Wire Line
+	8900 1175 8900 1275
+Connection ~ 8900 1175
+$Comp
+L power:GND #PWR0128
+U 1 1 5FFAFB5B
+P 8500 1875
+F 0 "#PWR0128" H 8500 1625 50  0001 C CNN
+F 1 "GND" H 8505 1702 50  0000 C CNN
+F 2 "" H 8500 1875 50  0001 C CNN
+F 3 "" H 8500 1875 50  0001 C CNN
+	1    8500 1875
+	1    0    0    -1
+$EndComp
+Connection ~ 9725 1250
+Wire Wire Line
+	9475 1250 9725 1250
+Wire Wire Line
+	9475 1050 9725 1050
+$Comp
+L Device:C_Small C25
+U 1 1 5FEC8637
+P 9475 1150
+F 0 "C25" H 9275 1200 50  0000 L CNN
+F 1 "4.7uF" H 9225 1100 50  0000 L CNN
+F 2 "Capacitor_SMD:C_0805_2012Metric" H 9475 1150 50  0001 C CNN
+F 3 "~" H 9475 1150 50  0001 C CNN
+	1    9475 1150
+	1    0    0    -1
+$EndComp
+$Comp
+L power:GND #PWR0155
+U 1 1 5FEC6232
+P 9725 1250
+F 0 "#PWR0155" H 9725 1000 50  0001 C CNN
+F 1 "GND" H 9730 1077 50  0000 C CNN
+F 2 "" H 9725 1250 50  0001 C CNN
+F 3 "" H 9725 1250 50  0001 C CNN
+	1    9725 1250
+	1    0    0    -1
+$EndComp
+$Comp
+L Device:C_Small C26
+U 1 1 5FEC6044
+P 9725 1150
+F 0 "C26" H 9817 1196 50  0000 L CNN
+F 1 "100nF" H 9817 1105 50  0000 L CNN
+F 2 "Capacitor_SMD:C_0603_1608Metric" H 9725 1150 50  0001 C CNN
+F 3 "~" H 9725 1150 50  0001 C CNN
+	1    9725 1150
+	1    0    0    -1
+$EndComp
+$Comp
+L Sensor_Pressure:LPS25HB U6
+U 1 1 6002FC1C
+P 8400 1375
+F 0 "U6" V 7833 1325 50  0000 C CNN
+F 1 "LPS25HB" V 7924 1325 50  0000 C CNN
+F 2 "Package_LGA:ST_HLGA-10_2.5x2.5mm_P0.6mm_LayoutBorder3x2y" H 8400 1175 50  0001 C CNN
+F 3 "www.st.com/resource/en/datasheet/lps25hb.pdf" H 8450 1025 50  0001 C CNN
+	1    8400 1375
+	0    1    1    0
+$EndComp
+Wire Wire Line
+	8800 1175 8900 1175
+Wire Wire Line
+	8800 1275 8900 1275
+$Comp
+L power:GND #PWR0129
+U 1 1 600485C8
+P 8300 1875
+F 0 "#PWR0129" H 8300 1625 50  0001 C CNN
+F 1 "GND" H 8275 1700 50  0000 C CNN
+F 2 "" H 8300 1875 50  0001 C CNN
+F 3 "" H 8300 1875 50  0001 C CNN
+	1    8300 1875
+	1    0    0    -1
+$EndComp
+$Comp
+L power:+3.3V #PWR0130
+U 1 1 6006B3D3
+P 9475 1050
+F 0 "#PWR0130" H 9475 900 50  0001 C CNN
+F 1 "+3.3V" H 9490 1223 50  0000 C CNN
+F 2 "" H 9475 1050 50  0001 C CNN
+F 3 "" H 9475 1050 50  0001 C CNN
+	1    9475 1050
+	1    0    0    -1
+$EndComp
+Connection ~ 9475 1050
+Wire Wire Line
+	1200 2800 1200 2825
+Wire Wire Line
+	1200 2800 1600 2800
+Connection ~ 1200 2800
+Connection ~ 1600 2800
 $EndSCHEMATC

Commit message: Layout + Routing v1 done
Connections:
- net GND: now also C36.2, C37.2
Changed lines of the file:
@@
 Connection ~ 1200 2800
 Connection ~ 1600 2800
+$Comp
+L power:GND #PWR?
+U 1 1 5FF89171
+P 6700 2675
+F 0 "#PWR?" H 6700 2425 50  0001 C CNN
+F 1 "GND" H 6825 2625 50  0000 C CNN
+F 2 "" H 6700 2675 50  0001 C CNN
+F 3 "" H 6700 2675 50  0001 C CNN
+	1    6700 2675
+	1    0    0    -1
+$EndComp
+Connection ~ 6700 2675
 $EndSCHEMATC

Commit message: Updated with final board design
Connections:
- net +3V3: now also U6.6 (~CS)
- net GND: no longer U6.6 (~CS)
Changed lines of the file:
@@
 	1    0    0    -1
 $EndComp
-Text GLabel 3750 1400 0    50   Input ~ 0
-FLASH_CS
 $Comp
 L power:+3.3V #PWR0161
@@
 	1    0    0    -1
 $EndComp
-Text GLabel 3750 1700 0    50   Input ~ 0
-SPI2_MOSI
-Text GLabel 3750 1800 0    50   Input ~ 0
-SPI2_MISO
-Text GLabel 3750 1500 0    50   Input ~ 0
-SPI2_SCK
 $Comp
 L RF_GPS:MAX-8Q U9
@@
 Wire Wire Line
 	1325 7150 1350 7150
+Wire Wire Line
+	8900 1175 8900 1275
+Connection ~ 8900 1175
+$Comp
+L power:GND #PWR0128
+U 1 1 5FFAFB5B
+P 8500 1875
+F 0 "#PWR0128" H 8500 1625 50  0001 C CNN
+F 1 "GND" H 8505 1702 50  0000 C CNN
+F 2 "" H 8500 1875 50  0001 C CNN
+F 3 "" H 8500 1875 50  0001 C CNN
+	1    8500 1875
+	1    0    0    -1
+$EndComp
+Connection ~ 9725 1250
+Wire Wire Line
+	9475 1250 9725 1250
+Wire Wire Line
+	9475 1050 9725 1050
+$Comp
+L Device:C_Small C25
+U 1 1 5FEC8637
+P 9475 1150
+F 0 "C25" H 9275 1200 50  0000 L CNN
+F 1 "4.7uF" H 9225 1100 50  0000 L CNN
+F 2 "Capacitor_SMD:C_0805_2012Metric" H 9475 1150 50  0001 C CNN
+F 3 "~" H 9475 1150 50  0001 C CNN
+	1    9475 1150
+	1    0    0    -1
+$EndComp
+$Comp
+L power:GND #PWR0155
+U 1 1 5FEC6232
+P 9725 1250
+F 0 "#PWR0155" H 9725 1000 50  0001 C CNN
+F 1 "GND" H 9730 1077 50  0000 C CNN
+F 2 "" H 9725 1250 50  0001 C CNN
+F 3 "" H 9725 1250 50  0001 C CNN
+	1    9725 1250
+	1    0    0    -1
+$EndComp
+$Comp
+L Device:C_Small C26
+U 1 1 5FEC6044
+P 9725 1150
+F 0 "C26" H 9817 1196 50  0000 L CNN
+F 1 "100nF" H 9817 1105 50  0000 L CNN
+F 2 "Capacitor_SMD:C_0603_1608Metric" H 9725 1150 50  0001 C CNN
+F 3 "~" H 9725 1150 50  0001 C CNN
+	1    9725 1150
+	1    0    0    -1
+$EndComp
+$Comp
+L Sensor_Pressure:LPS25HB U6
+U 1 1 6002FC1C
+P 8400 1375
+F 0 "U6" V 7833 1325 50  0000 C CNN
+F 1 "LPS25HB" V 7924 1325 50  0000 C CNN
+F 2 "Package_LGA:ST_HLGA-10_2.5x2.5mm_P0.6mm_LayoutBorder3x2y" H 8400 1175 50  0001 C CNN
+F 3 "www.st.com/resource/en/datasheet/lps25hb.pdf" H 8450 1025 50  0001 C CNN
+	1    8400 1375
+	0    1    1    0
+$EndComp
+Wire Wire Line
+	8800 1175 8900 1175
+Wire Wire Line
+	8800 1275 8900 1275
+$Comp
+L power:+3.3V #PWR0130
+U 1 1 6006B3D3
+P 9475 1050
+F 0 "#PWR0130" H 9475 900 50  0001 C CNN
+F 1 "+3.3V" H 9490 1223 50  0000 C CNN
+F 2 "" H 9475 1050 50  0001 C CNN
+F 3 "" H 9475 1050 50  0001 C CNN
+	1    9475 1050
+	1    0    0    -1
+$EndComp
+Connection ~ 9475 1050
+Wire Wire Line
+	1200 2800 1200 2825
+Wire Wire Line
+	1200 2800 1600 2800
+Connection ~ 1200 2800
+Connection ~ 1600 2800
+$Comp
+L power:GND #PWR0131
+U 1 1 5FF89171
+P 6700 2675
+F 0 "#PWR0131" H 6700 2425 50  0001 C CNN
+F 1 "GND" H 6825 2625 50  0000 C CNN
+F 2 "" H 6700 2675 50  0001 C CNN
+F 3 "" H 6700 2675 50  0001 C CNN
+	1    6700 2675
+	1    0    0    -1
+$EndComp
+Connection ~ 6700 2675
+$Comp
+L power:+3.3V #PWR0129
+U 1 1 5FF9862B
+P 8300 1875
+F 0 "#PWR0129" H 8300 1725 50  0001 C CNN
+F 1 "+3.3V" H 8350 2025 50  0000 C CNN
+F 2 "" H 8300 1875 50  0001 C CNN
+F 3 "" H 8300 1875 50  0001 C CNN
+	1    8300 1875
+	-1   0    0    1
+$EndComp
 $Comp
 L W25N01GVZEIG:W25N01GVZEIG_TR U5
@@
 	1    0    0    -1
 $EndComp
-Wire Wire Line
-	8900 1175 8900 1275
-Connection ~ 8900 1175
-$Comp
-L power:GND #PWR0128
-U 1 1 5FFAFB5B
-P 8500 1875
-F 0 "#PWR0128" H 8500 1625 50  0001 C CNN
-F 1 "GND" H 8505 1702 50  0000 C CNN
-F 2 "" H 8500 1875 50  0001 C CNN
-F 3 "" H 8500 1875 50  0001 C CNN
-	1    8500 1875
-	1    0    0    -1
-$EndComp
-Connection ~ 9725 1250
-Wire Wire Line
-	9475 1250 9725 1250
-Wire Wire Line
-	9475 1050 9725 1050
-$Comp
-L Device:C_Small C25
-U 1 1 5FEC8637
-P 9475 1150
-F 0 "C25" H 9275 1200 50  0000 L CNN
-F 1 "4.7uF" H 9225 1100 50  0000 L CNN
-F 2 "Capacitor_SMD:C_0805_2012Metric" H 9475 1150 50  0001 C CNN
-F 3 "~" H 9475 1150 50  0001 C CNN
-	1    9475 1150
-	1    0    0    -1
-$EndComp
-$Comp
-L power:GND #PWR0155
-U 1 1 5FEC6232
-P 9725 1250
-F 0 "#PWR0155" H 9725 1000 50  0001 C CNN
-F 1 "GND" H 9730 1077 50  0000 C CNN
-F 2 "" H 9725 1250 50  0001 C CNN
-F 3 "" H 9725 1250 50  0001 C CNN
-	1    9725 1250
-	1    0    0    -1
-$EndComp
-$Comp
-L Device:C_Small C26
-U 1 1 5FEC6044
-P 9725 1150
-F 0 "C26" H 9817 1196 50  0000 L CNN
-F 1 "100nF" H 9817 1105 50  0000 L CNN
-F 2 "Capacitor_SMD:C_0603_1608Metric" H 9725 1150 50  0001 C CNN
-F 3 "~" H 9725 1150 50  0001 C CNN
-	1    9725 1150
-	1    0    0    -1
-$EndComp
-$Comp
-L Sensor_Pressure:LPS25HB U6
-U 1 1 6002FC1C
-P 8400 1375
-F 0 "U6" V 7833 1325 50  0000 C CNN
-F 1 "LPS25HB" V 7924 1325 50  0000 C CNN
-F 2 "Package_LGA:ST_HLGA-10_2.5x2.5mm_P0.6mm_LayoutBorder3x2y" H 8400 1175 50  0001 C CNN
-F 3 "www.st.com/resource/en/datasheet/lps25hb.pdf" H 8450 1025 50  0001 C CNN
-	1    8400 1375
-	0    1    1    0
-$EndComp
-Wire Wire Line
-	8800 1175 8900 1175
-Wire Wire Line
-	8800 1275 8900 1275
-$Comp
-L power:GND #PWR0129
-U 1 1 600485C8
-P 8300 1875
-F 0 "#PWR0129" H 8300 1625 50  0001 C CNN
-F 1 "GND" H 8275 1700 50  0000 C CNN
-F 2 "" H 8300 1875 50  0001 C CNN
-F 3 "" H 8300 1875 50  0001 C CNN
-	1    8300 1875
-	1    0    0    -1
-$EndComp
-$Comp
-L power:+3.3V #PWR0130
-U 1 1 6006B3D3
-P 9475 1050
-F 0 "#PWR0130" H 9475 900 50  0001 C CNN
-F 1 "+3.3V" H 9490 1223 50  0000 C CNN
-F 2 "" H 9475 1050 50  0001 C CNN
-F 3 "" H 9475 1050 50  0001 C CNN
-	1    9475 1050
-	1    0    0    -1
-$EndComp
-Connection ~ 9475 1050
-Wire Wire Line
-	1200 2800 1200 2825
-Wire Wire Line
-	1200 2800 1600 2800
-Connection ~ 1200 2800
-Connection ~ 1600 2800
-$Comp
-L power:GND #PWR?
-U 1 1 5FF89171
-P 6700 2675
-F 0 "#PWR?" H 6700 2425 50  0001 C CNN
-F 1 "GND" H 6825 2625 50  0000 C CNN
-F 2 "" H 6700 2675 50  0001 C CNN
-F 3 "" H 6700 2675 50  0001 C CNN
-	1    6700 2675
-	1    0    0    -1
-$EndComp
-Connection ~ 6700 2675
+Text GLabel 3750 1500 0    50   Input ~ 0
+SPI2_SCK
+Text GLabel 3750 1800 0    50   Input ~ 0
+SPI2_MISO
+Text GLabel 3750 1700 0    50   Input ~ 0
+SPI2_MOSI
+Text GLabel 3750 1400 0    50   Input ~ 0
+FLASH_CS
 $EndSCHEMATC
