File: hardware/kiCad/Mercury/peripherals.sch (KiCad schematic (older format))
At the start: 48 parts, among them J13 5-1814832-1, J14 5-1814832-1, U4 MPU-6050, U5 W25N01GVZEIG_TR, U6 LPS25HB, U7 CC2500, U8 CC2592RGVR, U9 MAX-8Q, Y2 26 MHz Oscillator

Commit message: Sent For Manufacture
Parts:
- C19, C20, C21, C23, C27, C28, C29, C33: LCSC Part # (none) -> C1525
- C22: LCSC Part # (none) -> C1604
- C25: LCSC Part # (none) -> C1779
- C26: LCSC Part # (none) -> C14663
- C30, C31, C32: LCSC Part # (none) -> C1530
- C34, C35, C37, C40: LCSC Part # (none) -> C1547
- C36, C39: LCSC Part # (none) -> C1523
- C38, C45, C46: LCSC Part # (none) -> C52923
- C41, C42: LCSC Part # (none) -> C1559
- C43: LCSC Part # (none) -> C161338
- C44: LCSC Part # (none) -> C1549
- C47: LCSC Part # (none) -> C1567
- C48: LCSC Part # (none) -> C15195
- J13, J14: symbol SMA_ANT:5-1814832-1 -> Mercury-rescue:5-1814832-1-SMA_ANT
- L2: LCSC Part # (none) -> C13595
- L3: LCSC Part # (none) -> C18222
- L4: LCSC Part # (none) -> C18304
- L5: LCSC Part # (none) -> C18830
- R32, R33: LCSC Part # (none) -> C25900
- R34: LCSC Part # (none) -> C25796
- R35: LCSC Part # (none) -> C25118
- R36: LCSC Part # (none) -> C51721
- R37: LCSC Part # (none) -> C25744
- U4: LCSC Part # (none) -> C24112
- U5: symbol W25N01GVZEIG:W25N01GVZEIG_TR -> Mercury-rescue:W25N01GVZEIG_TR-W25N01GVZEIG; LCSC Part # (none) -> C88868
- U6: LCSC Part # (none) -> C87898
- U7: LCSC Part # (none) -> C57494
- U8: symbol CC2592:CC2592RGVR -> Mercury-rescue:CC2592RGVR-CC2592; LCSC Part # (none) -> C53274
- Y2: LCSC Part # (none) -> C23425
Connections:
- net +3V3: now also U6.6 (~CS)
- net GND: no longer U6.6 (~CS)
